Commit message: Added Seaos logo

File: tugbot_description/urdf/model.urdf (robot description, URDF)
Before this commit: robot tugbot, 10 links, 9 joints
Links:
- link base_link: geometry visual mesh ; visual mesh filename=file://

Commit message: for jazzy

File: tugbot_description/urdf/model.urdf (robot description, URDF)
Before this commit: robot tugbot, 10 links, 9 joints
Links:
- link base_link: geometry visual mesh filename=package://tugbot_description/meshes/base/movai-logo.png; visual mesh filename=package://tugbot_description/meshes/base/movai_logo.dae

Commit message: update seaos logo visulization on rviz2 and gazebo

File: tugbot_description/urdf/model.urdf (robot description, URDF)
Before this commit: robot tugbot, 10 links, 9 joints
Links:
- link base_link: geometry visual mesh filename=package://tugbot_description/meshes/base/movai_logo.dae; visual mesh filename=package://tugbot_description/meshes/base/seaos_logo.dae
